Commit message: Updated pkg to work with ros-noetic

File: my_model/urdf/robo_robot.urdf (robot description, URDF)
Before this commit: robot my_model, 7 links, 6 joints
Joints:
- joint left_wheel_joint: origin xyz=-0.03 -0.09 0 rpy=0 0 0 -> xyz=-0.03 0.09 0 rpy=0 0 0
- joint right_wheel_joint: origin xyz=-0.03 0.09 0 rpy=0 0 0 -> xyz=-0.03 -0.09 0 rpy=0 0 0

File: simbha_model/urdf/robo_robot.urdf (robot description, URDF)
Before this commit: robot simbha_model, 5 links, 4 joints
Joints:
- joint left_wheel_joint: origin xyz=-0.03 -0.09 0 rpy=0 0 0 -> xyz=-0.03 0.09 0 rpy=0 0 0
- joint right_wheel_joint: origin xyz=-0.03 0.09 0 rpy=0 0 0 -> xyz=-0.03 -0.09 0 rpy=0 0 0

File: simbha_model/urdf/simbha_robot.urdf (robot description, URDF)
Before this commit: robot simbha_model, 10 links, 9 joints
Joints:
- joint left_wheel_joint: origin xyz=0 -0.138 0.035 rpy=0 0 0 -> xyz=0 0.138 0.035 rpy=0 0 0
- joint right_wheel_joint: origin xyz=0.0 0.138 0.035 rpy=0 0 0 -> xyz=0.0 -0.138 0.035 rpy=0 0 0
